Commit message: fix sim

File: assets/robot/r1_pro/r1_pro.urdf (robot description, URDF)
Before this commit: robot R1_Pro, 49 links, 48 joints
Joints:
- joint torso_joint1: origin xyz=-0.032845 0 0.301 rpy=-1.5708 0 0 -> xyz=-0.032845 0 0.301 rpy=-1.5708 0.781000018119812 0; type revolute -> fixed
- joint torso_joint2: origin xyz=0 -0.4 0 rpy=0 0 0 -> xyz=0 -0.4 0 rpy=0 0 -1.7359000444412231; type revolute -> fixed
- joint torso_joint3: origin xyz=0 -0.3 0 rpy=0 0 0 -> xyz=0 -0.3 0 rpy=0 0 0.955; type revolute -> fixed
- joint torso_joint4: type revolute -> fixed
